File: Test.sch (KiCad schematic (older format))
At the start: 37 parts, among them P1 CONN_01X12, P10 CONN_01X12, P10a1 CONN_01X10, P11 CONN_01X03, P12 CONN_01X04, P13 CONN_02X04, P14 CONN_02X03, P15 CONN_02X05, P16 CONN_01X05, P17 CONN_01X01, P18 CONN_01X02, P19 CONN_01X08, P1a1 CONN_01X10, P2 CONN_01X12, P20 CONN_01X05, P21 CONN_01X05, P22 CONN_01X04, P23 CONN_01X04, P24 CONN_01X03, P25 CONN_01X10, P26 CONN_01X10, P27 CONN_01X10, P28 CONN_01X10, P2a1 CONN_01X10, P2a2 CONN_01X03, P2a3 CONN_01X03, P3 CONN_01X03, P4 CONN_01X24, P5 CONN_01X24, P6 CONN_01X03, P7 CONN_01X24, P8 CONN_01X24, P9 CONN_01X12, P9a1 CONN_01X10, SW1 SW_PUSH_SMALL_H, SW2 SW_PUSH_SMALL_H

Commit message: Version 2
Parts:
- removed P16: CONN_01X05, Socket_Strips:Socket_Strip_Straight_1x05, symbol CONN_01X05
- removed P24: CONN_01X03, Pin_Headers:Pin_Header_Straight_1x03, symbol CONN_01X03
- added P16: CONN_01X03, Socket_Strips:Socket_Strip_Straight_1x03, symbol CONN_01X03
- added P24: CONN_01X05, Pin_Headers:Pin_Header_Straight_1x05, symbol CONN_01X05
- P1, P10, P2, P9: value CONN_01X12 -> CONN_01X13; footprint Pin_Headers:Pin_Header_Straight_1x12 -> Pin_Headers:Pin_Header_Straight_1x13; symbol CONN_01X12 -> CONN_01X13
- P10a1: footprint Pin_Headers:Pin_Header_Straight_1x10 -> Pin_Headers:Pin_Header_Straight_1x09; symbol CONN_01X10 -> CONN_01X09
- P12: footprint Socket_Strips:Socket_Strip_Straight_1x04 -> Pin_Headers:Pin_Header_Straight_1x04
- P1a1, P2a1, P9a1: value CONN_01X10 -> CONN_01X09; footprint Pin_Headers:Pin_Header_Straight_1x10 -> Pin_Headers:Pin_Header_Straight_1x09; symbol CONN_01X10 -> CONN_01X09
- P21: footprint Pin_Headers:Pin_Header_Straight_1x05 -> Socket_Strips:Socket_Strip_Straight_1x05
- P22: footprint Pin_Headers:Pin_Header_Straight_1x04 -> Socket_Strips:Socket_Strip_Straight_1x04
Connections:
- net GND is gone; now on an unnamed net: P3.3 (P3)
- net at P2a2.1 (P1), P2a2.2 (P2), P2a2.3 (P3): now also P4.15 (P15), P5.15 (P15); no longer P4.14 (P14), P5.14 (P14)
- net at P7.1 (P1), P8.1 (P1): now also SW1.2, SW2.2
- net at P2a3.1 (P1), P2a3.2 (P2), P2a3.3 (P3): now also P7.15 (P15), P8.15 (P15); no longer P7.14 (P14), P8.14 (P14)
- net at P3.1 (P1): now also P18.1 (P1), P2.1 (P1), P2.10 (P10), P2.11 (P11), P2.12 (P12), P2.13 (P13), P2.2 (P2), P2.3 (P3), P2.4 (P4), P2.5 (P5), P2.6 (P6), P2.7 (P7), P2.8 (P8), P2.9 (P9), P26.1 (P1), P26.10 (P10), P26.2 (P2), P26.3 (P3), P26.4 (P4), P26.5 (P5), P26.6 (P6), P26.7 (P7), P26.8 (P8), P26.9 (P9), P28.1 (P1), P28.10 (P10), P28.2 (P2), P28.3 (P3), P28.4 (P4), P28.5 (P5), P28.6 (P6), P28.7 (P7), P28.8 (P8), P28.9 (P9), P2a1.1 (P1), P2a1.2 (P2), P2a1.3 (P3), P2a1.4 (P4), P2a1.5 (P5), P2a1.6 (P6), P2a1.7 (P7), P2a1.8 (P8), P2a1.9 (P9), P9.1 (P1), P9.10 (P10), P9.11 (P11), P9.12 (P12), P9.13 (P13), P9.2 (P2), P9.3 (P3), P9.4 (P4), P9.5 (P5), P9.6 (P6), P9.7 (P7), P9.8 (P8), P9.9 (P9), P9a1.1 (P1), P9a1.2 (P2), P9a1.3 (P3), P9a1.4 (P4), P9a1.5 (P5), P9a1.6 (P6), P9a1.7 (P7), P9a1.8 (P8), P9a1.9 (P9)
- net at P15.1 (P1): now also P20.5 (P5)
- net at P15.10 (P10): now also P24.5 (P5)
- net at P15.2 (P2): now also P24.1 (P1)
- net at P15.3 (P3): now also P20.4 (P4)
- net at P15.4 (P4): now also P24.2 (P2)
- net at P15.5 (P5): now also P20.3 (P3)
- net at P15.6 (P6): now also P24.3 (P3)
- net at P15.7 (P7): now also P20.2 (P2)
- net at P15.8 (P8): now also P24.4 (P4)
- net at P15.9 (P9): now also P20.1 (P1)
- net at P14.1 (P1): now also P6.3 (P3)
- net at P14.2 (P2): now also P16.1 (P1)
- net at P14.3 (P3): now also P6.2 (P2)
- net at P14.4 (P4): now also P16.2 (P2)
- net at P14.5 (P5): now also P6.1 (P1)
- net at P14.6 (P6): now also P16.3 (P3)
- net at P13.1 (P1): now also P12.4 (P4)
- net at P13.2 (P2): now also P19.4 (P4)
- net at P13.3 (P3): now also P12.3 (P3)
- net at P13.5 (P5): now also P12.2 (P2)
- net at P13.6 (P6): now also P19.6 (P6)
- net at P13.7 (P7): now also P12.1 (P1)
- net at P13.8 (P8): now also P19.7 (P7)
- net at P11.1 (P1): now also P19.3 (P3)
- net at P11.2 (P2): now also P19.2 (P2)
- net at P11.3 (P3): now also P19.1 (P1)
- net at P17.1 (P1): now also P18.2 (P2)
- net at BT1.1: now also P21.5 (P5)
- net at BT1.2: now also P1.1 (P1), P1.10 (P10), P1.11 (P11), P1.12 (P12), P1.13 (P13), P1.2 (P2), P1.3 (P3), P1.4 (P4), P1.5 (P5), P1.6 (P6), P1.7 (P7), P1.8 (P8), P1.9 (P9), P10.1 (P1), P10.10 (P10), P10.11 (P11), P10.12 (P12), P10.13 (P13), P10.2 (P2), P10.3 (P3), P10.4 (P4), P10.5 (P5), P10.6 (P6), P10.7 (P7), P10.8 (P8), P10.9 (P9), P10a1.1 (P1), P10a1.2 (P2), P10a1.3 (P3), P10a1.4 (P4), P10a1.5 (P5), P10a1.6 (P6), P10a1.7 (P7), P10a1.8 (P8), P10a1.9 (P9), P1a1.1 (P1), P1a1.2 (P2), P1a1.3 (P3), P1a1.4 (P4), P1a1.5 (P5), P1a1.6 (P6), P1a1.7 (P7), P1a1.8 (P8), P1a1.9 (P9), P25.1 (P1), P25.10 (P10), P25.2 (P2), P25.3 (P3), P25.4 (P4), P25.5 (P5), P25.6 (P6), P25.7 (P7), P25.8 (P8), P25.9 (P9), P27.1 (P1), P27.10 (P10), P27.2 (P2), P27.3 (P3), P27.4 (P4), P27.5 (P5), P27.6 (P6), P27.7 (P7), P27.8 (P8), P27.9 (P9)
- net at P22.1 (P1): now also P23.4 (P4)
- net at P22.2 (P2): now also P23.3 (P3)
- net at P22.3 (P3): now also P23.2 (P2)
- net at P22.4 (P4): now also P23.1 (P1)
- net at P21.1 (P1): now also SW1.1
- net at P21.2 (P2): now also SW2.1
- new net: P4.14 (P14), P5.14 (P14)
- new net: P7.14 (P14), P8.14 (P14)
Other:
- moved on the sheet: BT1, P11, P12, P13, P14, P15, P17, P18, P19, P20, P21, P22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
