File: Teensy_Uno/Teensy_Uno.sch (KiCad schematic (older format))
At the start: 30 parts, among them P1 Power, P10 CONN_01X13, P10a1 CONN_01X10, P11 CONN_01X24, P12 CONN_01X24, P13 CONN_01X05, P14 CONN_01X03, P15 CONN_01X03, P16 CONN_01X01, P17 CONN_01X24, P18 CONN_01X02, P19 CONN_01X24, P1a1 CONN_01X09, P2 Analog, P20 CONN_01X13, P21 CONN_01X13, P2a1 CONN_01X09, P3 Digital, P4 Digital, P5 CONN_01X01, P6 CONN_01X01, P7 CONN_01X01, P8 CONN_01X01, P9 CONN_01X13, P9a1 CONN_01X09, SW1 SW_PUSH_SMALL_H, SW2 SW_PUSH_SMALL_H

Commit message: fixed connection issues
Connections:
- net 12(MISO): now also P11.14 (P14), P12.14 (P14)
- net 2: no longer P11.4 (P4), P12.4 (P4), P4.6 (P6)
- new net: P11.4 (P4), P12.4 (P4), P4.6 (P6)
Changed lines of the file:
@@
 Text Label 5050 6050 0    60   ~ 0
 13(SCK)
+$Comp
+L R R1
+U 1 1 582628F2
+P 9700 6300
+F 0 "R1" V 9780 6300 50  0000 C CNN
+F 1 "10k" V 9700 6300 50  0000 C CNN
+F 2 "Resistors_ThroughHole:Resistor_Horizontal_RM10mm" V 9630 6300 50  0000 C CNN
+F 3 "" H 9700 6300 50  0000 C CNN
+	1    9700 6300
+	0    1    1    0
+$EndComp
+$Comp
+L R R2
+U 1 1 58262F0E
+P 9700 6600
+F 0 "R2" V 9780 6600 50  0000 C CNN
+F 1 "10k" V 9700 6600 50  0000 C CNN
+F 2 "Resistors_ThroughHole:Resistor_Horizontal_RM10mm" V 9630 6600 50  0000 C CNN
+F 3 "" H 9700 6600 50  0000 C CNN
+	1    9700 6600
+	0    1    1    0
+$EndComp
 Wire Wire Line
 	3300 5900 3300 6150
@@
 Wire Wire Line
 	4700 7350 5400 7350
-Wire Wire Line
-	4250 7250 5050 7250
 Wire Wire Line
 	4700 7150 7000 7150
@@
 	3950 3700 3950 4750
 Wire Wire Line
-	3900 4750 5800 4750
-Wire Wire Line
 	5850 6150 5850 4750
 Connection ~ 3250 3700
@@
 Wire Wire Line
 	7650 6350 8550 6350
-$Comp
-L R R1
-U 1 1 582628F2
-P 9700 6300
-F 0 "R1" V 9780 6300 50  0000 C CNN
-F 1 "10k" V 9700 6300 50  0000 C CNN
-F 2 "Resistors_ThroughHole:Resistor_Horizontal_RM10mm" V 9630 6300 50  0000 C CNN
-F 3 "" H 9700 6300 50  0000 C CNN
-	1    9700 6300
-	0    1    1    0
-$EndComp
-$Comp
-L R R2
-U 1 1 58262F0E
-P 9700 6600
-F 0 "R2" V 9780 6600 50  0000 C CNN
-F 1 "10k" V 9700 6600 50  0000 C CNN
-F 2 "Resistors_ThroughHole:Resistor_Horizontal_RM10mm" V 9630 6600 50  0000 C CNN
-F 3 "" H 9700 6600 50  0000 C CNN
-	1    9700 6600
-	0    1    1    0
-$EndComp
 Wire Wire Line
 	8850 6350 9550 6350
@@
 Wire Wire Line
 	9850 6300 9850 6600
+Wire Wire Line
+	5850 4750 3950 4750
+Wire Wire Line
+	4250 7250 4700 7250
 $EndSCHEMATC

Commit message: corrected reset voltage to 3.3v
Connections:
- net at P1.4 (P4), P11.15 (P15), P12.15 (P15): now also R1.1, R2.1
- net at P16.1 (P1), P18.2 (P2): no longer R1.1, R2.1
Changed lines of the file:
@@
 	2750 3900 3250 3900
 Wire Wire Line
-	2750 3800 3250 3800
+	2750 3800 3650 3800
 Wire Wire Line
 	2750 3700 3950 3700
@@
 	9550 6650 9550 6600
 Wire Wire Line
-	7800 1350 7800 2000
-Wire Wire Line
-	7800 2000 10450 2000
-Wire Wire Line
-	10450 2000 10450 6300
-Wire Wire Line
 	10450 6300 9850 6300
 Wire Wire Line
@@
 Wire Wire Line
 	4250 7250 4700 7250
+Wire Wire Line
+	10450 6300 10450 4950
+Wire Wire Line
+	10450 4950 3650 4950
+Wire Wire Line
+	3650 4950 3650 3800
+Connection ~ 3250 3800
 $EndSCHEMATC

Commit message: Additional corrections
Parts:
- removed R1, R2: 10k, Resistors_ThroughHole:Resistor_Horizontal_RM10mm, symbol R
Connections:
- net A0: now also P17.13 (P13), P19.13 (P13)
- net at P1.4 (P4), P11.15 (P15): no longer P12.15 (P15)
- net at BT1.2, P1.6 (P6), P1.7 (P7)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: now also P10a1.1 (P1), P10a1.2 (P2), P10a1.3 (P3), P10a1.4 (P4), P10a1.5 (P5), P10a1.6 (P6), P10a1.7 (P7), P10a1.8 (P8), P10a1.9 (P9), P15.3 (P3), P21.1 (P1), P21.10 (P10), P21.11 (P11), P21.12 (P12), P21.13 (P13), P21.2 (P2), P21.3 (P3), P21.4 (P4), P21.5 (P5), P21.6 (P6), P21.7 (P7), P21.8 (P8), P21.9 (P9), SW1.2, SW2.2
Changed lines of the file:
@@
 Text Label 5050 6050 0    60   ~ 0
 13(SCK)
-$Comp
-L R R1
-U 1 1 582628F2
-P 9700 6300
-F 0 "R1" V 9780 6300 50  0000 C CNN
-F 1 "10k" V 9700 6300 50  0000 C CNN
-F 2 "Resistors_ThroughHole:Resistor_Horizontal_RM10mm" V 9630 6300 50  0000 C CNN
-F 3 "" H 9700 6300 50  0000 C CNN
-	1    9700 6300
-	0    1    1    0
-$EndComp
-$Comp
-L R R2
-U 1 1 58262F0E
-P 9700 6600
-F 0 "R2" V 9780 6600 50  0000 C CNN
-F 1 "10k" V 9700 6600 50  0000 C CNN
-F 2 "Resistors_ThroughHole:Resistor_Horizontal_RM10mm" V 9630 6600 50  0000 C CNN
-F 3 "" H 9700 6600 50  0000 C CNN
-	1    9700 6600
-	0    1    1    0
-$EndComp
 Wire Wire Line
 	3300 5900 3300 6150
@@
 	8000 3650 9050 3650
 Wire Wire Line
-	8500 3550 8000 3550
+	7150 3550 8500 3550
 Wire Wire Line
 	7050 3350 8500 3350
@@
 	2750 3900 3250 3900
 Wire Wire Line
-	2750 3800 3650 3800
-Wire Wire Line
 	2750 3700 3950 3700
 Wire Wire Line
@@
 	2750 2500 3750 2500
 Wire Wire Line
-	2750 2400 3250 2400
+	2750 2400 3300 2400
 Connection ~ 9350 3750
 Connection ~ 9350 3850
@@
 	5050 4250 5300 4250
 Connection ~ 5300 4250
-Connection ~ 6200 1100
 Connection ~ 6400 1100
 Wire Wire Line
@@
 Wire Wire Line
 	6400 1800 1750 1800
-Wire Wire Line
-	9950 750  6200 750
-Wire Wire Line
-	6200 750  6200 1100
 Connection ~ 2750 2400
 Connection ~ 7800 1350
@@
 Connection ~ 1750 2300
 Connection ~ 9350 2300
-Connection ~ 9950 2300
 Wire Wire Line
 	9350 2300 8500 2300
@@
 	8500 2300 8500 2350
 Wire Wire Line
-	2750 2400 2750 2050
-Wire Wire Line
 	2750 2050 1150 2050
 Wire Wire Line
@@
 	9350 1100 9350 5950
 Wire Wire Line
-	9950 750  9950 4550
+	9950 750  9950 4950
 Wire Wire Line
 	7350 1350 7350 1950
@@
 Connection ~ 3250 2500
 Wire Wire Line
-	7900 3550 7150 3550
-Wire Wire Line
 	7150 3550 7150 1700
 Wire Wire Line
@@
 	8850 6350 9550 6350
 Wire Wire Line
-	9550 6350 9550 6300
-Wire Wire Line
-	8850 6650 9550 6650
-Wire Wire Line
-	9550 6650 9550 6600
+	9850 6650 8850 6650
 Wire Wire Line
 	10450 6300 9850 6300
 Wire Wire Line
-	9850 6300 9850 6600
+	9850 6300 9850 6650
 Wire Wire Line
 	5850 4750 3950 4750
@@
 Wire Wire Line
 	10450 6300 10450 4950
-Wire Wire Line
-	10450 4950 3650 4950
-Wire Wire Line
-	3650 4950 3650 3800
 Connection ~ 3250 3800
+Wire Wire Line
+	10450 4950 9950 4950
+Connection ~ 9950 2300
+Connection ~ 6200 1100
+Wire Wire Line
+	6200 750  6200 1100
+Wire Wire Line
+	9950 750  6200 750
+Wire Wire Line
+	2750 2050 2750 2400
+Wire Wire Line
+	6200 1100 3300 1100
+Wire Wire Line
+	3300 1100 3300 2400
+Connection ~ 3250 2400
+Connection ~ 8000 3550
+Wire Wire Line
+	9550 6350 9550 6650
+Connection ~ 9550 6650
 $EndSCHEMATC
