File: Teensy 35 Breakout v2/Teensy 35 Breakout v2.kicad_pcb (KiCad board)
At the start: 2 copper layers, 99.1 x 106.7 mm, 41 parts, among them P1 CONN_01X13, P10 CONN_01X13, P10a1 CONN_01X10, P11 CONN_01X03, P12 CONN_01X04, P13 CONN_02X04, P14 CONN_02X03, P15 CONN_02X05, P16 CONN_01X03, P17 CONN_01X01, P18 CONN_01X02, P19 CONN_01X08, P1a1 CONN_01X09, P2 CONN_01X13, P20 CONN_01X05, P21 CONN_01X05, P22 CONN_01X04, P23 CONN_01X04, P24 CONN_01X05, P25 CONN_01X10, P26 CONN_01X10, P27 CONN_01X10, P28 CONN_01X10, P2a1 CONN_01X09, P2a2 CONN_01X03, P2a3 CONN_01X03, P3 CONN_01X03, P4 CONN_01X24, P5 CONN_01X24, P6 CONN_01X03, P7 CONN_01X24, P8 CONN_01X24, P9 CONN_01X13, P9a1 CONN_01X09, SW1 SW_PUSH_SMALL_H, SW2 SW_PUSH_SMALL_H

Commit message: Final updates and corrections
Parts:
- moved P27 5.59 mm to (129.8, 116.3)
- moved P28 5.59 mm to (129.8, 120.1)
- moved P25 5.59 mm to (73.9, 116.3)
- moved P26 5.59 mm to (73.9, 120.1)
- moved SW1 5.59 mm to (106.9, 118.9)
- moved SW2 5.59 mm to (118.4, 118.9)
- moved REF3 5.14 mm to (70.1, 126.5)
- moved RE4 4.64 mm to (154.4, 126.2)
- moved REF2 4.26 mm to (71.4, 47.0)
- moved P20 2.29 mm to (76.2, 99.3)
Routing:
- net Net-(P21-Pad1): track 49.0 -> 35.3 mm
- net Net-(P18-Pad1): track 278.8 -> 267.1 mm
- net Net-(BT1-Pad1): track 85.4 -> 75.6 mm
- net Net-(BT1-Pad2): track 271.0 -> 261.7 mm
- net Net-(P2a3-Pad1): track 74.8 -> 68.6 mm
- net Net-(P21-Pad2): track 34.7 -> 30.2 mm
- net Net-(P7-Pad1): track 1.19 -> 2.88 mm
- net Net-(P15-Pad1): track 36.6 -> 37.3 mm
Other:
- board size 99.1 x 106.7 mm -> 93 x 99.6 mm

Commit message: Correcyrf some connections
Routing:
- net Net-(BT1-Pad2): track 261.7 -> 275.3 mm
- net Net-(P18-Pad1): track 267.1 -> 276.8 mm
- net Net-(P7-Pad1): track 2.88 -> 1.71 mm
Changed lines of the file:
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@@
     (thickness 1.6)
     (drawings 29)
-    (tracks 414)
+    (tracks 426)
     (zones 0)
     (modules 41)
@@
   (segment (start 93.3926 62.2691) (end 93.3926 46.4026) (width 0.25) (layer F.Cu) (net 1))
   (segment (start 103.514 72.39) (end 93.3926 62.2691) (width 0.25) (layer F.Cu) (net 1))
+  (segment (start 96.774 116.332) (end 99.314 116.332) (width 0.25) (layer B.Cu) (net 2))
+  (segment (start 99.314 116.332) (end 101.092 118.11) (width 0.25) (layer B.Cu) (net 2))
+  (segment (start 101.092 118.11) (end 101.092 123.19) (width 0.25) (layer B.Cu) (net 2))
+  (segment (start 101.092 123.19) (end 102.362 124.46) (width 0.25) (layer B.Cu) (net 2))
+  (segment (start 102.362 124.46) (end 122.936 124.46) (width 0.25) (layer B.Cu) (net 2))
+  (segment (start 122.936 124.46) (end 125.73 121.666) (width 0.25) (layer B.Cu) (net 2))
+  (segment (start 125.73 121.666) (end 125.73 117.856) (width 0.25) (layer B.Cu) (net 2))
+  (segment (start 125.73 117.856) (end 127.254 116.332) (width 0.25) (layer B.Cu) (net 2))
+  (segment (start 127.254 116.332) (end 129.794 116.332) (width 0.25) (layer B.Cu) (net 2))
+  (segment (start 96.774 116.332) (end 96.774 117.598) (width 0.25) (layer B.Cu) (net 2))
   (segment (start 138.349 38.1) (end 137.16 38.1) (width 0.25) (layer F.Cu) (net 2))
   (segment (start 138.349 52.07) (end 138.349 38.1) (width 0.25) (layer F.Cu) (net 2))
@@
   (segment (start 85.09 109.22) (end 85.09 106.68) (width 0.25) (layer F.Cu) (net 2))
   (segment (start 132.334 116.332) (end 129.794 116.332) (width 0.25) (layer B.Cu) (net 2))
-  (segment (start 128.605 116.332) (end 129.794 116.332) (width 0.25) (layer B.Cu) (net 2))
-  (segment (start 127.577 117.36) (end 128.605 116.332) (width 0.25) (layer B.Cu) (net 2))
-  (segment (start 98.9914 117.36) (end 127.577 117.36) (width 0.25) (layer B.Cu) (net 2))
-  (segment (start 97.9629 116.332) (end 98.9914 117.36) (width 0.25) (layer B.Cu) (net 2))
   (segment (start 96.774 116.332) (end 97.9629 116.332) (width 0.25) (layer B.Cu) (net 2))
   (segment (start 96.774 116.332) (end 94.234 116.332) (width 0.25) (layer B.Cu) (net 2))
@@
   (segment (start 85.09 110.409) (end 85.1765 110.4956) (width 0.25) (layer F.Cu) (net 2))
   (segment (start 85.09 109.22) (end 85.09 110.409) (width 0.25) (layer F.Cu) (net 2))
+  (segment (start 96.774 120.142) (end 99.314 120.142) (width 0.25) (layer B.Cu) (net 3))
+  (segment (start 99.314 120.142) (end 99.822 120.65) (width 0.25) (layer B.Cu) (net 3))
+  (segment (start 99.822 120.65) (end 99.822 124.714) (width 0.25) (layer B.Cu) (net 3))
+  (segment (start 99.822 124.714) (end 101.6 126.492) (width 0.25) (layer B.Cu) (net 3))
+  (segment (start 101.6 126.492) (end 124.968 126.492) (width 0.25) (layer B.Cu) (net 3))
+  (segment (start 124.968 126.492) (end 129.794 121.666) (width 0.25) (layer B.Cu) (net 3))
+  (segment (start 129.794 121.666) (end 129.794 120.142) (width 0.25) (layer B.Cu) (net 3))
   (segment (start 136.559 41.91) (end 147.32 41.91) (width 0.25) (layer B.Cu) (net 3))
   (segment (start 133.269 38.6201) (end 136.559 41.91) (width 0.25) (layer B.Cu) (net 3))
@@
   (segment (start 135.89 81.28) (end 135.89 78.74) (width 0.25) (layer F.Cu) (net 3))
   (segment (start 135.89 109.22) (end 135.89 106.68) (width 0.25) (layer F.Cu) (net 3))
-  (segment (start 129.794 120.142) (end 96.774 120.142) (width 0.25) (layer B.Cu) (net 3))
   (segment (start 87.803 107.95) (end 87.884 108.031) (width 0.25) (layer F.Cu) (net 3))
   (segment (start 87.63 107.95) (end 87.803 107.95) (width 0.25) (layer F.Cu) (net 3))
@@
   (segment (start 136.144 120.142) (end 136.144 110.825) (width 0.25) (layer F.Cu) (net 3))
   (segment (start 121.562 51.9889) (end 120.731 52.8197) (width 0.25) (layer F.Cu) (net 3))
+  (segment (start 120.731 52.8197) (end 119.9 51.9889) (width 0.25) (layer F.Cu) (net 3))
   (segment (start 90.17 86.36) (end 92.71 86.36) (width 0.25) (layer B.Cu) (net 4))
   (segment (start 104.14 86.36) (end 97.79 86.36) (width 0.25) (layer B.Cu) (net 4))
@@
   (segment (start 119.38 51.9889) (end 119.38 50.8) (width 0.25) (layer F.Cu) (net 87))
   (segment (start 119.9 51.9889) (end 119.38 51.9889) (width 0.25) (layer F.Cu) (net 87))
-  (segment (start 120.731 52.8197) (end 119.9 51.9889) (width 0.25) (layer F.Cu) (net 87))
 )

Commit message: update
Parts:
- added P29: USB_A, Connect:USB_A, F.Cu at (110.2, 45.1)
- P22: value CONN_01X04 -> CONN_01X05; footprint Socket_Strips:Socket_Strip_Straight_1x04 -> Socket_Strips:Socket_Strip_Straight_1x05
- P23: value CONN_01X04 -> CONN_01X05; footprint Pin_Headers:Pin_Header_Straight_1x04 -> Pin_Headers:Pin_Header_Straight_1x05
- moved P22 2.29 mm to (108.0, 57.4)
- moved REF2 1.14 mm to (70.9, 46.0)
Connections:
- P23 pad 1: Net-(P22-Pad4) -> Net-(P22-Pad5)
- P23 pad 2: Net-(P22-Pad3) -> Net-(P22-Pad4)
- P23 pad 3: Net-(P22-Pad2) -> Net-(P22-Pad3)
- P23 pad 4: Net-(P22-Pad1) -> Net-(P22-Pad2)
Routing:
- net Net-(P22-Pad5): track 0.00 -> 75.7 mm
- net Net-(P22-Pad4): track 35.1 -> 58.1 mm
- net Net-(P12-Pad4): track 63.2 -> 42.8 mm
- net Net-(P22-Pad3): track 35.1 -> 54.5 mm
- net Net-(P22-Pad1): track 35.1 -> 52.7 mm
- net Net-(P22-Pad2): track 35.1 -> 52.4 mm
Other:
- board text added: "24 25 26 27 28 29 30"
- board text added: "A12/R4 A13/T4"
- board text added: "A22 A21 A20 SDA1 SCL1 A17 A16 RX5 TX5"
- board text added: "A24 A23 48 47 3.3v"
- board text added: "A9 A8 A7 A6 SCL0 SDA0 A3 A2 A1 A0/K0 SCK0"
- board text added: "GND RX1 TX1 2 SCL2 SDA2 5 6"
- board text added: "RX3 TX3 RX2 CS0 MOSI0 MISO0"
- board text added: "T3.5 A26 A25 Gnd Gnd"
- board text added: "T3.6 5V DP DM Gnd Gnd"
- board text removed: "A12 A13"
- board text removed: "A24 A23 SDA0 SCL0 3.3v"
- board text removed: "A26 A25 Gnd Gnd"
- board text removed: "A9 A8 A7 A6 SCL0 SDA0 A3 A2 A1 A0"
- board text removed: "DAC1 DAC0 A20 SDA1 SCL1 A17 A16 RX5 TX5"
- board text removed: "GND"
- board text removed: "RX1 TX1 SCL2 SDA2"
- board text removed: "RX3 TX3 RX2 TX2"
