File: Teensy 35 Breakout v2/Teensy 35 Breakout v2.sch (KiCad schematic (older format))
At the start: 37 parts, among them P1 CONN_01X13, P10 CONN_01X13, P10a1 CONN_01X10, P11 CONN_01X03, P12 CONN_01X04, P13 CONN_02X04, P14 CONN_02X03, P15 CONN_02X05, P16 CONN_01X03, P17 CONN_01X01, P18 CONN_01X02, P19 CONN_01X08, P1a1 CONN_01X09, P2 CONN_01X13, P20 CONN_01X05, P21 CONN_01X05, P22 CONN_01X04, P23 CONN_01X04, P24 CONN_01X05, P25 CONN_01X10, P26 CONN_01X10, P27 CONN_01X10, P28 CONN_01X10, P2a1 CONN_01X09, P2a2 CONN_01X03, P2a3 CONN_01X03, P3 CONN_01X03, P4 CONN_01X24, P5 CONN_01X24, P6 CONN_01X03, P7 CONN_01X24, P8 CONN_01X24, P9 CONN_01X13, P9a1 CONN_01X09, SW1 SW_PUSH_SMALL_H, SW2 SW_PUSH_SMALL_H

Commit message: update
Parts:
- added P29: USB_A, Connect:USB_A, symbol USB_A
- P22: value CONN_01X04 -> CONN_01X05; footprint Socket_Strips:Socket_Strip_Straight_1x04 -> Socket_Strips:Socket_Strip_Straight_1x05; symbol CONN_01X04 -> CONN_01X05
- P23: value CONN_01X04 -> CONN_01X05; footprint Pin_Headers:Pin_Header_Straight_1x04 -> Pin_Headers:Pin_Header_Straight_1x05; symbol CONN_01X04 -> CONN_01X05
Connections:
- net at P22.1 (P1): now also P23.5 (P5), P29.1 (VCC); no longer P23.4 (P4)
- net at P22.2 (P2): now also P23.4 (P4), P29.2 (D-); no longer P23.3 (P3)
- net at P22.3 (P3): now also P23.3 (P3), P29.3 (D+); no longer P23.2 (P2)
- net at P22.4 (P4): now also P23.2 (P2), P29.4 (GND); no longer P23.1 (P1)
- new net: P22.5 (P5), P23.1 (P1), P29.5 (shield)
Changed lines of the file:
@@
 LIBS:contrib
 LIBS:valves
-LIBS:Teensy 35 Breakout v1-cache
+LIBS:Teensy 35 Breakout v2-cache
 EELAYER 25 0
 EELAYER END
@@
 $EndComp
 $Comp
-L CONN_01X04 P22
+L CONN_01X05 P22
 U 1 1 57F9BE0A
-P 4750 2300
-F 0 "P22" H 4750 2550 50  0000 C CNN
-F 1 "CONN_01X04" V 4850 2300 50  0000 C CNN
-F 2 "Socket_Strips:Socket_Strip_Straight_1x04" H 4750 2300 50  0001 C CNN
-F 3 "" H 4750 2300 50  0000 C CNN
-	1    4750 2300
-	1    0    0    -1
-$EndComp
-$Comp
-L CONN_01X04 P23
+P 4750 2250
+F 0 "P22" H 4750 2500 50  0000 C CNN
+F 1 "CONN_01X05" V 4850 2250 50  0000 C CNN
+F 2 "Socket_Strips:Socket_Strip_Straight_1x05" H 4750 2250 50  0001 C CNN
+F 3 "" H 4750 2250 50  0000 C CNN
+	1    4750 2250
+	1    0    0    -1
+$EndComp
+$Comp
+L CONN_01X05 P23
 U 1 1 57F9D60A
-P 4000 2300
-F 0 "P23" H 4000 2550 50  0000 C CNN
-F 1 "CONN_01X04" V 4100 2300 50  0000 C CNN
-F 2 "Pin_Headers:Pin_Header_Straight_1x04" H 4000 2300 50  0001 C CNN
-F 3 "" H 4000 2300 50  0000 C CNN
-	1    4000 2300
+P 4000 2250
+F 0 "P23" H 4000 2500 50  0000 C CNN
+F 1 "CONN_01X05" V 4100 2250 50  0000 C CNN
+F 2 "Pin_Headers:Pin_Header_Straight_1x05" H 4000 2250 50  0001 C CNN
+F 3 "" H 4000 2250 50  0000 C CNN
+	1    4000 2250
 	-1   0    0    1
 $EndComp
@@
 	4200 2150 4550 2150
 Wire Wire Line
-	4550 2250 4200 2250
-Wire Wire Line
-	4200 2350 4550 2350
+	4200 2250 4550 2250
+Wire Wire Line
+	4200 2350 4600 2350
 Wire Wire Line
 	4550 2450 4200 2450
@@
 	7000 4750 7000 3850
 Connection ~ 7800 3850
+Wire Wire Line
+	4200 2050 4550 2050
+Connection ~ 4200 2050
+Connection ~ 4550 2050
+$Comp
+L USB_A P29
+U 1 1 586306D0
+P 4500 1250
+F 0 "P29" H 4700 1050 50  0000 C CNN
+F 1 "USB_A" H 4450 1450 50  0000 C CNN
+F 2 "Connect:USB_A" V 4450 1150 50  0001 C CNN
+F 3 "" V 4450 1150 50  0000 C CNN
+	1    4500 1250
+	1    0    0    -1
+$EndComp
+Wire Wire Line
+	4550 2050 4550 1800
+Wire Wire Line
+	4550 1800 4300 1800
+Wire Wire Line
+	4300 1800 4300 1550
+Wire Wire Line
+	4400 2150 4400 1550
+Wire Wire Line
+	4500 2250 4500 1550
+Wire Wire Line
+	4600 2350 4600 1550
+Connection ~ 4300 1550
+Connection ~ 4400 1550
+Connection ~ 4500 1550
+Connection ~ 4600 1550
+Connection ~ 4400 2150
+Connection ~ 4500 2250
+Wire Wire Line
+	4550 2450 4550 2600
+Wire Wire Line
+	4550 2600 5000 2600
+Wire Wire Line
+	5000 2600 5000 1150
+Wire Wire Line
+	5000 1150 4800 1150
+Connection ~ 4800 1150
 $EndSCHEMATC
