File: PropShield_Uno/PropShield_Uno.kicad_pcb (KiCad board)
At the start: 2 copper layers, 68.6 x 53.3 mm, 19 parts, among them J1 CONN_01X14, J10 CONN_01X02, J2 CONN_01X04, J3 CONN_01X05, J4 CONN_01X04, J5 CONN_01X14, J6 CONN_01X04, J7 CONN_01X04, J8 CONN_01X02, J9 CONN_01X03, P1 Power, P2 Analog, P3 Digital, P4 Digital, P5 CONN_01X01, P6 CONN_01X01, P7 CONN_02X03

Commit message: Design Update
Parts:
- D3, D4: value D_Schottky_ALT -> D_Schottky; footprint Diodes_SMD:D_SOD-323 -> Diodes_THT:D_DO-15_P10.16mm_Horizontal
- moved D3 1.10 mm to (154.9, 112.8)
- moved J2 0.99 mm to (172.7, 99.3)
Routing:
- net /A4(SDA): track 71.5 -> 111.9 mm
- net Net-(D4-Pad2): track 33.1 -> 49.0 mm
- net /6(**): track 37.9 -> 51.2 mm
- net /12(MISO): track 53.9 -> 42.7 mm
- net /5(**): track 42.3 -> 53.0 mm
- net /2: track 48.1 -> 58.1 mm, vias 1 -> 0
- net Net-(J2-Pad2): track 68.3 -> 61.9 mm, vias 0 -> 1
- net +5V: track 15.3 -> 20.8 mm
- net Net-(D3-Pad1): track 108.1 -> 113.4 mm
- net /A5(SCL): track 77.2 -> 73.0 mm, vias 0 -> 1
- net Net-(J2-Pad3): track 63.2 -> 59.8 mm, vias 0 -> 1
- net /7: track 32.5 -> 30.9 mm, vias 0 -> 1
- net Net-(J2-Pad4): track 58.1 -> 59.4 mm
- net Net-(J10-Pad2): track 59.7 -> 61.0 mm
- net Net-(J3-Pad5): track 93.9 -> 95.2 mm, vias 1 -> 0
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