File: PropShield_Uno/PropShield_Uno.sch (KiCad schematic (older format))
At the start: 16 parts, among them J1 CONN_01X14, J10 CONN_01X02, J2 CONN_01X04, J3 CONN_01X05, J4 CONN_01X04, J5 CONN_01X14, J6 CONN_01X04, J7 CONN_01X04, J8 CONN_01X02, J9 CONN_01X03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

Commit message: Design Update
Parts:
- D3, D4: value D_Schottky_ALT -> D_Schottky; footprint Diodes_SMD:D_SOD-323 -> Diodes_THT:D_DO-15_P10.16mm_Horizontal; symbol D_Schottky_ALT -> D_Schottky
Changed lines of the file:
@@
 $EndComp
 $Comp
-L D_Schottky_ALT D3
+L D_Schottky D3
 U 1 1 5939B1F1
 P 5000 6400
 F 0 "D3" H 5000 6500 50  0000 C CNN
-F 1 "D_Schottky_ALT" H 5000 6300 50  0000 C CNN
-F 2 "Diodes_SMD:D_SOD-323" H 5000 6400 50  0001 C CNN
+F 1 "D_Schottky" H 5000 6300 50  0000 C CNN
+F 2 "Diodes_THT:D_DO-15_P10.16mm_Horizontal" H 5000 6400 50  0001 C CNN
 F 3 "" H 5000 6400 50  0001 C CNN
 	1    5000 6400
@@
 $EndComp
 $Comp
-L D_Schottky_ALT D4
+L D_Schottky D4
 U 1 1 5939BBC9
 P 5750 7000
 F 0 "D4" H 5750 7100 50  0000 C CNN
-F 1 "D_Schottky_ALT" H 5750 6900 50  0000 C CNN
-F 2 "Diodes_SMD:D_SOD-323" H 5750 7000 50  0001 C CNN
+F 1 "D_Schottky" H 5750 6900 50  0000 C CNN
+F 2 "Diodes_THT:D_DO-15_P10.16mm_Horizontal" H 5750 7000 50  0001 C CNN
 F 3 "" H 5750 7000 50  0001 C CNN
 	1    5750 7000
 	1    0    0    -1
 $EndComp
+Text Label 7700 3800 0    60   ~ 0
+GND
 Wire Wire Line
 	4650 3700 4650 3950
@@
 	6900 4500 6900 4800
 Connection ~ 7400 4800
-Wire Wire Line
-	6550 4400 7000 4400
-Wire Wire Line
-	7000 4400 7000 4700
-Connection ~ 7400 4700
 Wire Wire Line
 	6550 4300 7050 4300
@@
 Connection ~ 6850 6150
 Connection ~ 5400 6400
-Text Label 7700 3800 0    60   ~ 0
-GND
+Connection ~ 7400 4700
+Wire Wire Line
+	6550 4400 7000 4400
+Wire Wire Line
+	7000 4400 7000 4700
 $EndSCHEMATC
